File: pulses_plus_submin_panel.kicad_pcb (KiCad board)
At the start: 2 copper layers, 40.2 x 128.5 mm, 27 parts

Commit message: Make pulses_plus_submin footprint and 3D refs portable
The project had two references that only resolved on the machine it was
authored on:

- Thonkiconn_PJ301M.kicad_mod pointed its 3D model at
  ${KIPRJMOD}/SW-T2-4E-B-A2-MA2/3D/..., a directory that does not exist.
  The model is actually in 3d/, so repoint it there.

- pulses_plus_submin_panel.kicad_pcb placed 27 footprints from a "Panel"
  library that is in neither the project fp-lib-table nor the tree; it
  resolved from a KiCad global table locally, so the panel would not open
  on a fresh clone. Vendor its three footprints (Hole_3.2mm, Hole_4.95mm,
  Hole_6mm -- each a single NPTH circular pad) into
  pulses_plus_submin.pretty and rewrite the refs to pulses_plus_submin:.

Both boards now resolve entirely from KiCad stock libraries plus this
project's own ${KIPRJMOD}-relative library and 3D models.

The vendored footprints keep the placed instances' "Rescue" pad layer
rather than the conventional *.Mask, so board and library agree exactly
and the already-fabbed gerbers are unchanged; see the footprint descr
for why not to "fix" it.

Verified with kicad-cli 10.0.0: panel DRC returns its pre-existing 66
violations with zero library errors (was 27 lib_footprint_issues before,
27 lib_footprint_mismatch mid-way); main board unchanged at 1
pre-existing text_height; STEP export completes with no missing models.

Co-Authored-By: Claude Opus 5 <noreply@anthropic.com>
Parts:
- ? (x14): footprint Panel:Hole_3.2mm -> pulses_plus_submin:Hole_3.2mm
- ? (x10): footprint Panel:Hole_4.95mm -> pulses_plus_submin:Hole_4.95mm
- ? (x3): footprint Panel:Hole_6mm -> pulses_plus_submin:Hole_6mm
Changed lines of the file:
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@@
 		)
 	)
-	(footprint "Panel:Hole_3.2mm"
+	(footprint "pulses_plus_submin:Hole_3.2mm"
 		(layer "F.Cu")
 		(at 119.34 37.907)
@@
 		(embedded_fonts no)
 	)
-	(footprint "Panel:Hole_4.95mm"
+	(footprint "pulses_plus_submin:Hole_4.95mm"
 		(layer "F.Cu")
 		(at 119.64 132.482)
@@
 		(embedded_fonts no)
 	)
-	(footprint "Panel:Hole_4.95mm"
+	(footprint "pulses_plus_submin:Hole_4.95mm"
 		(layer "F.Cu")
 		(at 144.2 74.807)
@@
 		(embedded_fonts no)
 	)
-	(footprint "Panel:Hole_4.95mm"
+	(footprint "pulses_plus_submin:Hole_4.95mm"
 		(layer "F.Cu")
 		(at 119.64 98.807)
@@
 		(embedded_fonts no)
 	)
-	(footprint "Panel:Hole_3.2mm"
+	(footprint "pulses_plus_submin:Hole_3.2mm"
 		(layer "F.Cu")
 		(at 131.92 96.307)
@@
 		(embedded_fonts no)
 	)
-	(footprint "Panel:Hole_4.95mm"
+	(footprint "pulses_plus_submin:Hole_4.95mm"
 		(layer "F.Cu")
 		(at 144.2 58.807)
@@
 		(embedded_fonts no)
 	)
-	(footprint "Panel:Hole_4.95mm"
+	(footprint "pulses_plus_submin:Hole_4.95mm"
 		(layer "F.Cu")
 		(at 119.64 66.807)
@@
 		(embedded_fonts no)
 	)
-	(footprint "Panel:Hole_6mm"
+	(footprint "pulses_plus_submin:Hole_6mm"
 		(layer "F.Cu")
 		(at 144.2 146.332)
@@
 		(embedded_fonts no)
 	)
-	(footprint "Panel:Hole_3.2mm"
+	(footprint "pulses_plus_submin:Hole_3.2mm"
 		(layer "F.Cu")
 		(at 131.92 72.307)
@@
 		(embedded_fonts no)
 	)
-	(footprint "Panel:Hole_3.2mm"
+	(footprint "pulses_plus_submin:Hole_3.2mm"
 		(layer "F.Cu")
 		(at 119.64 122.6)
@@
 		(embedded_fonts no)
 	)
-	(footprint "Panel:Hole_3.2mm"
+	(footprint "pulses_plus_submin:Hole_3.2mm"
 		(layer "F.Cu")
 		(at 131.92 56.307)
@@
 		(embedded_fonts no)
 	)
-	(footprint "Panel:Hole_3.2mm"
+	(footprint "pulses_plus_submin:Hole_3.2mm"
 		(layer "F.Cu")
 		(at 144.5 160.407)
@@
 		(embedded_fonts no)
 	)
-	(footprint "Panel:Hole_3.2mm"
+	(footprint "pulses_plus_submin:Hole_3.2mm"
 		(layer "F.Cu")
 		(at 144.5 37.907)
@@
 		(embedded_fonts no)
 	)
-	(footprint "Panel:Hole_3.2mm"
+	(footprint "pulses_plus_submin:Hole_3.2mm"
 		(layer "F.Cu")
 		(at 119.34 160.407)
@@
 		(embedded_fonts no)
 	)
-	(footprint "Panel:Hole_3.2mm"
+	(footprint "pulses_plus_submin:Hole_3.2mm"
 		(layer "F.Cu")
 		(at 131.92 88.307)
@@
 		(embedded_fonts no)
 	)
-	(footprint "Panel:Hole_4.95mm"
+	(footprint "pulses_plus_submin:Hole_4.95mm"
 		(layer "F.Cu")
 		(at 119.64 82.807)
@@
 		(embedded_fonts no)
 	)
-	(footprint "Panel:Hole_4.95mm"
+	(footprint "pulses_plus_submin:Hole_4.95mm"
 		(layer "F.Cu")
 		(at 119.64 50.807)
@@
 		(embedded_fonts no)
 	)
-	(footprint "Panel:Hole_3.2mm"
+	(footprint "pulses_plus_submin:Hole_3.2mm"
 		(layer "F.Cu")
 		(at 131.92 104.307)
@@
 		(embedded_fonts no)
 	)
-	(footprint "Panel:Hole_6mm"
+	(footprint "pulses_plus_submin:Hole_6mm"
 		(layer "F.Cu")
 		(at 119.64 146.332)
@@
 		(embedded_fonts no)
 	)
-	(footprint "Panel:Hole_4.95mm"
+	(footprint "pulses_plus_submin:Hole_4.95mm"
 		(layer "F.Cu")
 		(at 144.2 132.482)
@@
 		(embedded_fonts no)
 	)
-	(footprint "Panel:Hole_4.95mm"
+	(footprint "pulses_plus_submin:Hole_4.95mm"
 		(layer "F.Cu")
 		(at 144.2 106.807)
@@
 		(embedded_fonts no)
 	)
-	(footprint "Panel:Hole_3.2mm"
+	(footprint "pulses_plus_submin:Hole_3.2mm"
 		(layer "F.Cu")
 		(at 131.92 64.307)
@@
 		(embedded_fonts no)
 	)
-	(footprint "Panel:Hole_6mm"
+	(footprint "pulses_plus_submin:Hole_6mm"
 		(layer "F.Cu")
 		(at 119.64 112.243)
@@
 		(embedded_fonts no)
 	)
-	(footprint "Panel:Hole_3.2mm"
+	(footprint "pulses_plus_submin:Hole_3.2mm"
 		(layer "F.Cu")
 		(at 131.92 48.307)
@@
 		(embedded_fonts no)
 	)
-	(footprint "Panel:Hole_3.2mm"
+	(footprint "pulses_plus_submin:Hole_3.2mm"
 		(layer "F.Cu")
 		(at 144.2 122.6)
@@
 		(embedded_fonts no)
 	)
-	(footprint "Panel:Hole_3.2mm"
+	(footprint "pulses_plus_submin:Hole_3.2mm"
 		(layer "F.Cu")
 		(at 131.92 80.307)
@@
 		(embedded_fonts no)
 	)
-	(footprint "Panel:Hole_4.95mm"
+	(footprint "pulses_plus_submin:Hole_4.95mm"
 		(layer "F.Cu")
 		(at 144.2 90.807)
