File: pulses_plus_submin_panel_v2.kicad_pcb (KiCad board)
At the start: 2 copper layers, 40.2 x 128.5 mm, 27 parts

Commit message: Keep the NonCommercial clause: CC BY-NC-SA 4.0 on the panel back
The v2 panel back read CC-BY-SA, which is a different licence from the
CC BY-NC-SA 4.0 the v1 panel carries -- it would have permitted commercial
builds of the module. Restores the NC clause and the version number.

PANEL_STYLE goes to v1.04: the licence line now has to be the short form
*with* its version, and says why the clause letters are not cosmetic.

Co-Authored-By: Claude Opus 5 <noreply@anthropic.com>
Other:
- board text added: "."
Changed lines of the file:
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@@
 	)
 	(gr_text "C"
-		(at 136.9950 152.9070)
+		(at 142.0700 152.9070)
 		(layer "B.SilkS")
 		(effects
@@
 	)
 	(gr_text "C"
-		(at 135.5450 152.9070)
+		(at 140.6200 152.9070)
+		(layer "B.SilkS")
+		(effects
+			(font
+				(size 1.35 1.35)
+				(thickness 0.25)
+			)
+			(justify mirror)
+		)
+	)
+	(gr_text "B"
+		(at 137.7200 152.9070)
+		(layer "B.SilkS")
+		(effects
+			(font
+				(size 1.35 1.35)
+				(thickness 0.25)
+			)
+			(justify mirror)
+		)
+	)
+	(gr_text "Y"
+		(at 136.2700 152.9070)
 		(layer "B.SilkS")
 		(effects
@@
 	)
 	(gr_text "-"
-		(at 134.0950 152.9070)
+		(at 134.8200 152.9070)
 		(layer "B.SilkS")
 		(effects
@@
 		)
 	)
-	(gr_text "B"
-		(at 132.6450 152.9070)
+	(gr_text "N"
+		(at 133.3700 152.9070)
 		(layer "B.SilkS")
 		(effects
@@
 		)
 	)
-	(gr_text "Y"
-		(at 131.1950 152.9070)
+	(gr_text "C"
+		(at 131.9200 152.9070)
 		(layer "B.SilkS")
 		(effects
@@
 	)
 	(gr_text "-"
-		(at 129.7450 152.9070)
+		(at 130.4700 152.9070)
 		(layer "B.SilkS")
 		(effects
@@
 	)
 	(gr_text "S"
-		(at 128.2950 152.9070)
+		(at 129.0200 152.9070)
 		(layer "B.SilkS")
 		(effects
@@
 	)
 	(gr_text "A"
-		(at 126.8450 152.9070)
+		(at 127.5700 152.9070)
 		(layer "B.SilkS")
 		(effects
+			(font
+				(size 1.35 1.35)
+				(thickness 0.25)
+			)
+			(justify mirror)
+		)
+	)
+	(gr_text "4"
+		(at 124.6700 152.9070)
+		(layer "B.SilkS")
+		(effects
+			(font
+				(size 1.35 1.35)
+				(thickness 0.25)
+			)
+			(justify mirror)
+		)
+	)
+	(gr_text "."
+		(at 123.2200 152.9070)
+		(layer "B.SilkS")
+		(effects
+			(font
+				(size 1.35 1.35)
+				(thickness 0.25)
+			)
+			(justify mirror)
+		)
+	)
+	(gr_text "0"
+		(at 121.7700 152.9070)
+		(layer "B.SilkS")
+		(effects

Commit message: v2 panel: standard mounting slots, copper decoration redrawn as silk
Mounting is regenerated to the house rule instead of inherited. 8 HP is
> 6 HP, so both columns and four 6.4 x 3.2 mm obround slots milled on
Edge.Cuts, horizontal so the module can slide +/- 1.6 mm onto the rails.
Centres sit 3.0 mm from the top and bottom edges; the 7.5 mm inset is the
datum and the far column steps out 5 x 5.08 to 32.9, leaving a 7.26 mm
margin on that side -- the grid is what the rail is drilled to, so that is
the way round that matters. The four round 3.2 mm holes are gone.

The decorative copper is gone with them: all 29 track segments deleted and
the zones' cached fills dropped, since those fills flowed around tracks that
no longer exist and would otherwise plot as ghost clearances. Zones refill
from scratch on open.

What the copper was saying is now said in silkscreen at LINE_W, per the wire
rule -- one knee, 0/90/45 only, stopping short of what it joins:

- each toggle to its indicator LED, leaving clear of the throw mark
- the EXT jack to channel 8, which is what it normals into
- bus indicator to mode switch, and mode switch to output jack, as two runs
  rather than one: a single wire would cross the mode switch, and a wire may
  not cross a control

The title refits to 2.8 mm: a milled slot edge is a board edge, so the title
now has to hold EDGE_MARGIN off it as well as off the first LED hole, and the
band that leaves is 6.0 mm for two lines.

kicad-cli 10.0.0 DRC: 0 violations, down from 66. All 23 control holes remain
byte-identical to v1.

Co-Authored-By: Claude Opus 5 <noreply@anthropic.com>
Parts:
- removed the ? at (119.3, 37.9)
- removed the ? at (144.5, 160.4)
- removed the ? at (144.5, 37.9)
- removed the ? at (119.3, 160.4)
Routing:
- net (no net): track 198.4 -> 0.00 mm
Other:
- outline, holes or cut-outs redrawn
